File: Hardware/Logic_Level_Converter.brd (EAGLE design)
At the start: 15.2 x 12.7 mm, 17 parts, among them Q1 BSS138, Q2 BSS138

Commit message: Resistor Value Changes and  Revision Code Update
Changed the vales of r5 and r9 resistors from 10k to 20k.  Added the
revision # to the schematic.
Parts:
- R5, R9: value 10K -> 20K
Changed lines of the file:
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@@
 <attribute name="VALUE" x="7.366" y="7.493" size="0.4064" layer="27" rot="R90"/>
 </element>
-<element name="R5" library="SparkFun" package="0603-RES" value="10K" x="6.35" y="4.699" smashed="yes" rot="R90">
+<element name="R5" library="SparkFun" package="0603-RES" value="20K" x="6.35" y="4.699" smashed="yes" rot="R90">
 <attribute name="NAME" x="5.6515" y="3.81" size="0.4064" layer="25" rot="R90"/>
 <attribute name="VALUE" x="7.366" y="4.191" size="0.4064" layer="27" rot="R90"/>
@@
 <attribute name="VALUE" x="8.382" y="7.493" size="0.4064" layer="27" rot="R90"/>
 </element>
-<element name="R9" library="SparkFun" package="0603-RES" value="10K" x="8.89" y="4.699" smashed="yes" rot="R90">
+<element name="R9" library="SparkFun" package="0603-RES" value="20K" x="8.89" y="4.699" smashed="yes" rot="R90">
 <attribute name="NAME" x="8.1915" y="3.81" size="0.4064" layer="25" rot="R90"/>
 <attribute name="VALUE" x="8.382" y="4.191" size="0.4064" layer="27" rot="R90"/>

Commit message: Updated Voltage Table / Added Creative Commons/Rev
Changed the Example Voltage table to reflect the new resistor values as
well as added an equation for reference.  Added the creative commons
license and designed by/revised by names.
Parts:
- added CC_TEXT1: CREATIVE_COMMONS, SparkFun-Aesthetics:CREATIVE_COMMONS
Other:
- board text added: "Nathan Seidle"
- board text added: "Rev V13 by Patrick Alberts"
